File: HackPad1.kicad_pcb (KiCad board)
At the start: 2 copper layers, 60 x 60 mm, 9 parts, among them SW1 SW_SPDT, U1 ATtiny85V-10P

Commit message: updated design basics
Routing:
- net GND: track 103.4 -> 85.1 mm
- net +3.3V: track 75.3 -> 74.4 mm
- added copper zone on B.Cu, net GND
- removed copper zone on F.Cu, net GND
Changed lines of the file:
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@@
-	)
-	(segment
-		(start 117.23 98.5)
-		(end 117.23 98.27)
-		(width 0.5)
-		(layer "F.Cu")
-		(net 2)
 	)
 	(segment
@@
 	)
 	(segment
-		(start 117.23 98.02)
-		(end 133 82.25)
-		(width 0.5)
-		(layer "B.Cu")
-		(net 2)
-	)
-	(segment
-		(start 133 82.25)
-		(end 131.4 82.25)
-		(width 0.5)
-		(layer "B.Cu")
-		(net 2)
-	)
-	(segment
 		(start 147.12 69)
 		(end 138.82 60.7)
@@
 	)
 	(segment
+		(start 143.367767 82.25)
+		(end 131.4 82.25)
+		(width 0.5)
+		(layer "B.Cu")
+		(net 2)
+	)
+	(segment
 		(start 131.4 82.25)
 		(end 130.15 81)
@@
 	)
 	(segment
-		(start 143.367767 82.25)
-		(end 133 82.25)
-		(width 0.5)
-		(layer "B.Cu")
-		(net 2)
-	)
-	(segment
-		(start 117.23 98.5)
-		(end 117.23 98.02)
+		(start 117.23 96.42)
+		(end 131.4 82.25)
 		(width 0.5)
 		(layer "B.Cu")
@@
 	)
 	(segment
+		(start 117.23 98.5)
+		(end 117.23 96.42)
+		(width 0.5)
+		(layer "B.Cu")
+		(net 2)
+	)
+	(segment
 		(start 145 84.105)
 		(end 146.665 85.77)
@@
 	)
 	(segment
+		(start 140.029999 67.03)
+		(end 138.302233 67.03)
+		(width 0.5)
+		(layer "F.Cu")
+		(net 6)
+	)
+	(segment
+		(start 141.4 68.400001)
+		(end 140.029999 67.03)
+		(width 0.5)
+		(layer "F.Cu")
+		(net 6)
+	)
+	(segment
+		(start 137.57 62.722233)
+		(end 138.302233 61.99)
+		(width 0.5)
+		(layer "F.Cu")
+		(net 6)
+	)
+	(segment
+		(start 138.302233 67.03)
+		(end 137.57 66.297767)
+		(width 0.5)
+		(layer "F.Cu")
+		(net 6)
+	)
+	(segment
+		(start 141.4 73.55)
+		(end 141.4 68.400001)
+		(width 0.5)
+		(layer "F.Cu")
+		(net 6)
+	)
+	(segment
+		(start 139.337767 61.99)
+		(end 159 81.652233)
+		(width 0.5)
+		(layer "F.Cu")
+		(net 6)
+	)
+	(segment
+		(start 137.57 66.297767)
+		(end 137.57 62.722233)
+		(width 0.5)
+		(layer "F.Cu")
+		(net 6)
+	)
+	(segment
+		(start 159 81.652233)
+		(end 159 82.8)
+		(width 0.5)
+		(layer "F.Cu")
+		(net 6)
+	)
+	(segment
+		(start 138.302233 61.99)
+		(end 139.337767 61.99)
+		(width 0.5)
+		(layer "F.Cu")
+		(net 6)
+	)
+	(segment
 		(start 116.5 76.55)
 		(end 116.5 75.5)
@@
 	)
 	(segment
-		(start 137.88 75)
-		(end 131.2 68.32)
-		(width 0.5)
-		(layer "F.Cu")
-		(net 6)
-	)
-	(segment
-		(start 142.85 75)
-		(end 137.88 75)
-		(width 0.5)
-		(layer "F.Cu")
-		(net 6)
-	)
-	(segment
-		(start 112.65 80.4)
-		(end 113.9 80.4)
-		(width 0.5)
-		(layer "F.Cu")
-		(net 6)
-	)
-	(segment
 		(start 112.65 80.4)
 		(end 116.5 76.55)
@@
 	)
 	(segment
-		(start 140.387767 60.5)
-		(end 137.887767 58)
-		(width 0.5)
-		(layer "B.Cu")
+		(start 142.85 75)
+		(end 141.4 73.55)
+		(width 0.5)
+		(layer "F.Cu")
 		(net 6)
 	)
 	(segment
 		(start 124.02 75.5)
-		(end 126.76 72.76)
-		(width 0.5)
-		(layer "B.Cu")
-		(net 6)
-	)
-	(segment
-		(start 158.08 81.88)
-		(end 158.08 69.962233)
+		(end 131.2 68.32)
 		(width 0.5)
 		(layer "B.Cu")
@@
 	)
 	(segment
-		(start 128 58)
-		(end 126.76 59.24)
-		(width 0.5)
-		(layer "B.Cu")
-		(net 6)
-	)
-	(segment
-		(start 137.887767 58)
-		(end 128 58)
-		(width 0.5)
-		(layer "B.Cu")
-		(net 6)
-	)
-	(segment
-		(start 126.76 59.24)
-		(end 126.76 72.76)
-		(width 0.5)
-		(layer "B.Cu")
-		(net 6)
-	)
-	(segment
-		(start 148.617767 60.5)
-		(end 140.387767 60.5)
-		(width 0.5)
-		(layer "B.Cu")
-		(net 6)
-	)
-	(segment
-		(start 126.76 72.76)
-		(end 131.2 68.32)
-		(width 0.5)
-		(layer "B.Cu")
-		(net 6)
-	)
-	(segment
-		(start 158.08 69.962233)
-		(end 148.617767 60.5)
-		(width 0.5)
-		(layer "B.Cu")
-		(net 6)
-	)
-	(segment
-		(start 159 82.8)
-		(end 158.08 81.88)
+		(start 131.2 68.32)
+		(end 137.88 75)
+		(width 0.5)
+		(layer "B.Cu")
+		(net 6)
+	)
+	(segment
+		(start 137.88 75)
+		(end 142.85 75)
 		(width 0.5)
 		(layer "B.Cu")
@@
 		(net 6)
 		(net_name "GND")
-		(layer "F.Cu")
+		(layer "B.Cu")
 		(hatch edge 0.5)
 		(connect_pads
@@
 		(polygon
 			(pts
-				(xy 137 54) (xy 156 59) (xy 164 73) (xy 165 93) (xy 158 105.5) (xy 148 113.5) (xy 122.5 118.5) (xy 113.5 111.5)
-				(xy 107.5 103) (xy 137.5 54) (xy 137 53.5)
+				(xy 106 68.5) (xy 121 54) (xy 143 53.5) (xy 157 63.5) (xy 164.5 77.5) (xy 163.5 93) (xy 153 111.5)
+				(xy 128.5 118) (xy 107 107.5) (xy 102 91.5) (xy 102.5 75.5) (xy 106.5 68)
 			)
 		)
-	)
-	(zone
-		(net 6)
-		(net_name "GND")
-		(layer "F.Cu")
-		(hatch edge 0.5)
-		(priority 1)
-		(connect_pads
-			(clearance 0.5)
-		)
-		(min_thickness 0.25)
-		(filled_areas_thickness no)
-		(fill
-			(thermal_gap 0.5)
-			(thermal_bridge_width 0.5)
-		)
-		(polygon
-			(pts
-				(xy 96.5 67) (xy 139 51.5) (xy 97.5 65) (xy 97 67)
-			)
-		)
