File: _autosave-HackPad1.kicad_pcb (KiCad board)
At the start: 2 copper layers, 3.6 x 3.3 mm, 30 parts, among them J1 Conn_01x04_Pin, SW1 SW_Push, SW10 RotaryEncoder, SW2 SW_Push, SW3 SW_Push, SW4 SW_Push, SW5 SW_Push, SW6 SW_Push, SW7 SW_Push, SW8 SW_Push, SW9 SW_Push, U1 MOUDLE-SEEEDUINO-XIAO

Commit message: updated LED schematic(switched from 9 to 4)
Parts:
- moved D13 131.5 mm to (81.7, 134.2), turned to 90 degrees
- moved D10 114.4 mm to (81.8, 114.0), turned to 90 degrees
- moved D11 110.7 mm to (101.8, 114.0), turned to 90 degrees
- moved D12 89.8 mm to (121.1, 113.7), turned to 90 degrees
