File: _autosave-HackPad1.kicad_pcb (KiCad board)
At the start: 2 copper layers, 79 x 89 mm, 25 parts, among them J1 Conn_01x04_Pin, SW1 SW_Push, SW10 RotaryEncoder, SW2 SW_Push, SW3 SW_Push, SW4 SW_Push, SW5 SW_Push, SW6 SW_Push, SW7 SW_Push, SW8 SW_Push, SW9 SW_Push, U1 MOUDLE-SEEEDUINO-XIAO

Commit message: completed pcb design
Parts:
- moved D11 0.60 mm to (121.7, 114.2)
Routing:
- net GND: track 166.5 -> 13.0 mm, vias 1 -> 2
- net ENCA: track 66.6 -> 73.3 mm
- net Net-(D12-DOUT): track 31.2 -> 37.8 mm
- net +5V: track 122.9 -> 118.3 mm, vias 3 -> 1
- net COL2: track 91.1 -> 93.5 mm
- net ROW1: track 82.9 -> 84.8 mm, vias 1 -> 0
- net ENCB: track 57.3 -> 58.3 mm
- net Net-(D10-DOUT): track 20.0 -> 20.6 mm
- net Net-(D11-DOUT): track 16.7 -> 16.4 mm, vias 2 -> 0
- net COL3: track 118.1 -> 117.9 mm, vias 1 -> 0
- added copper zone on B.Cu, net GND
